File: bye_big/bye_big.sch (KiCad schematic (older format))
At the start: 22 parts, among them Q1 PZT2222A, SW1 SW_Push, U1 ATtiny85V-10PU, U2 MC78L05_SOT89, Y1 Resonator

Commit message: bye_big: FIX gnd not connected on uC
Connections:
- net gnd: now also U1.4 (GND)
Changed lines of the file:
@@
 Wire Wire Line
 	2950 5400 3350 5400
+Text GLabel 4050 3500 2    50   Input ~ 0
+gnd
+Wire Wire Line
+	4050 3400 4050 3500
 $EndSCHEMATC
