File: bye_big/bye_big.kicad_pcb (KiCad board)
At the start: 2 copper layers, 55.4 x 31.2 mm, 22 parts, among them Q1 PZT2222A, SW1 SW_Push, U1 ATtiny85V-10PU, U2 MC78L05_SOT89, Y1 Resonator

Commit message: bye_big: FIX gnd not connected on uC
Connections:
- U1 pad 4: (no net) -> gnd

Commit message: update to kicad 7
Other:
- net class Default removed

Commit message: add 7.0 files, fix missing symbols
Parts:
- C1: value CP -> C_Polarized
- U1: value ATtiny85V-10PU -> ATtiny85V-10P
Changed lines of the file:
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@@
     (property "Sheetfile" "bye_big.kicad_sch")
     (property "Sheetname" "")
+    (property "ki_description" "Polarized capacitor")
+    (property "ki_keywords" "cap capacitor")
     (attr smd)
     (fp_text reference "C1" (at 0 -4.35) (layer "F.SilkS")
         (effects (font (size 1 1) (thickness 0.15)))
     )
-    (fp_text value "CP" (at 0 4.35) (layer "F.Fab")
+    (fp_text value "C_Polarized" (at 0 4.35) (layer "F.Fab")
         (effects (font (size 1 1) (thickness 0.15)))
     )
@@
     (property "Sheetfile" "bye_big.kicad_sch")
     (property "Sheetname" "")
+    (property "ki_description" "10MHz, 8kB Flash, 512B SRAM, 512B EEPROM, debugWIRE, DIP-8")
+    (property "ki_keywords" "AVR 8bit Microcontroller tinyAVR")
     (attr through_hole)
     (fp_text reference "U1" (at 3.81 -2.33 90) (layer "F.SilkS")
         (effects (font (size 1 1) (thickness 0.15)))
     )
-    (fp_text value "ATtiny85V-10PU" (at 3.81 9.95 90) (layer "F.Fab")
-        (effects (font (size 1 1) (thickness 0.15)))
-    )
+    (fp_text value "ATtiny85V-10P" (at 3.81 9.95 90) (layer "F.Fab")
+        (effects (font (size 1 1) (thickness 0.15)))
+    )
